Commit message: change dummy_link to base_footprint

File: src/follow_me_py/urdf/tracer_mini.urdf (robot description, URDF)
Before this commit: robot tracer_mini, 9 links, 8 joints
Links:
- removed link dummy_link
- added link base_footprint
Joints:
- joint dummy_to_base: parent dummy_link -> base_footprint
